Commit message: fix direction bugs

File: src/agv_description/urdf/agv_base.urdf (robot description, URDF)
Before this commit: robot agv, 6 links, 5 joints
Links:
- link agv_link: mass 4.0 -> None; geometry collision mesh filename=package://agv_description/meshes/agv_base/agv_center.STL; visual mesh filename=package://agv_description/meshes/agv_base/agv_center.STL
